Commit message: robot model in Gazebo with changing the tires into cylinders + until the plug in

File: urdf/rabe_bot_basic.urdf.xacro (robot description, xacro)
@@ -8,5 +8,5 @@
                               <origin xyz="0.0 0.0 0.0" rpy="0.0 0.0 0.0"/>
                               <mass value="0.5"/>
-                              <inertia ixx="0.0" ixy="0.0" ixz="0.0" iyy="0.0" iyz="0.0" izz="0.0"/>
+                              <inertia ixx="0.4" ixy="0.0" ixz="0.0" iyy="0.4" iyz="0.0" izz="0.2"/>
                     </inertial>
                     <visual name="">
@@ -85,5 +85,5 @@
                               <origin xyz="0.0 0.0 0.0" rpy="0.0 0.0 0.0"/>
                               <mass value="0.2"/>
-                              <inertia ixx="0.0" ixy="0.0" ixz="0.0" iyy="0.0" iyz="0.0" izz="0.0"/>
+                              <inertia ixx="0.4" ixy="0.0" ixz="0.0" iyy="0.4" iyz="0.0" izz="0.2"/>
                     </inertial>
                     <visual name="">
@@ -111,6 +111,6 @@
                     <limit lower="0.0" upper="0.0" effort="0.0" velocity="0.0"/>
           </joint>
-          <!--right front wheel-->
-          <xacro:macro name="wheel" params="name x y">
+          <!-- right front wheel -->
+          <xacro:macro name="wheel_right" params="name x y">
                <link name="${name}_link">
                               <inertial>
@@ -122,5 +122,6 @@
                                         <origin xyz="0.0 0.0 0.0" rpy="0.0 0.0 0.0"/>
                                         <geometry>
-                                                  <mesh filename="package://robot_simulation_description/meshes/left1_tire.stl" scale="0.005 0.005 0.005"/>
+                                             <cylinder radius="0.15" length="0.1"/>
+                                             <!-- <mesh filename="package://robot_simulation_description/meshes/left1_tire.stl" scale="0.005 0.005 0.005"/> -->
                                         </geometry>
                                         <material name="black">
@@ -132,13 +133,14 @@
                                         <origin xyz="0.0 0.0 0.0" rpy="0.0 0.0 0.0"/>
                                         <geometry>
-                                                  <mesh filename="package://robot_simulation_description/meshes/left1_tire.stl" scale="0.005 0.005 0.005"/>
+                                             <cylinder radius="0.15" length="0.1"/>
+                                             <!-- <mesh filename="package://robot_simulation_description/meshes/left1_tire.stl" scale="0.005 0.005 0.005"/> -->
                                         </geometry>
                               </collision>
                     </link>
                     <joint name="${name}_joint" type="continuous">
-                              <origin xyz="${x} ${y} 0.0" rpy=" 0.0 1.57 0.0 "/>
+                              <origin xyz="${x} ${y} 0.0" rpy="0.0 1.5705 1.5705 "/>
                               <parent link="base_link"/>
                               <child link="${name}_link"/>
-                              <axis xyz="0.0 1.0 0.0"/>
+                              <axis xyz="0.0 0.0 1.0"/>
                     </joint>
           </xacro:macro>
@@ -153,5 +155,6 @@
                                         <origin xyz="0.0 0.0 0.0" rpy="0.0 0.0 0.0"/>
                                         <geometry>
-                                             <mesh filename="package://robot_simulation_description/meshes/right1_tire.stl" scale="0.005 0.005 0.005"/>
+                                             <cylinder radius="0.15" length="0.1"/>
+                                             <!-- <mesh filename="package://robot_simulation_description/meshes/right1_tire.stl" scale="0.005 0.005 0.005"/> -->
                                         </geometry>
                                         <material name="black">
@@ -163,18 +166,19 @@
                                         <origin xyz="0.0 0.0 0.0" rpy="0.0 0.0 0.0"/>
                                         <geometry>
-                                             <mesh filename="package://robot_simulation_description/meshes/right1_tire.stl" scale="0.005 0.005 0.005"/>
+                                             <cylinder radius="0.15" length="0.1"/>
+                                             <!-- <mesh filename="package://robot_simulation_description/meshes/right1_tire.stl" scale="0.005 0.005 0.005"/> -->
                                         </geometry>
                               </collision>
                     </link>
                     <joint name="${name}_joint" type="continuous">
-                              <origin xyz="${x} ${y} 0.0" rpy=" 0.0 1.57 0.0 "/>
+                              <origin xyz="${x} ${y} 0.0" rpy="0.0 1.5705 1.5705 "/>
                               <parent link="base_link"/>
                               <child link="${name}_link"/>
-                              <axis xyz="0.0 1.0 0.0"/>
+                              <axis xyz="0.0 0.0 1.0"/>
                     </joint>
           </xacro:macro>
-<xacro:wheel name="front_right_wheel" x="0.2" y="-0.26"/>
+<xacro:wheel_right name="front_right_wheel" x="0.2" y="-0.26"/>
 <xacro:wheel_left name="front_left_wheel" x="0.2" y="0.26"/>
-<xacro:wheel name="rear_right_wheel" x="-0.2" y="-0.26"/>
+<xacro:wheel_right name="rear_right_wheel" x="-0.2" y="-0.26"/>
 <xacro:wheel_left name="rear_left_wheel" x="-0.2" y="0.26"/>
 </robot>

Commit message: robot model in Gazebo with Kinect and LiDAR camera but not their plug in inside Gazebo yet

File: urdf/rabe_bot_basic.urdf.xacro (robot description, xacro)
@@ -182,3 +182,63 @@
 <xacro:wheel_right name="rear_right_wheel" x="-0.2" y="-0.26"/>
 <xacro:wheel_left name="rear_left_wheel" x="-0.2" y="0.26"/>
+          <!---Kinect/Depth Camera-->
+          <link name="camera_link">
+               <inertial>
+                    <origin xyz="0.0 0.0 0.0" rpy="0.0 0.0 0.0"/>
+                    <mass value="0.1"/>
+                    <inertia ixx="0.0" ixy="0.0" ixz="0.0" iyy="0.0" iyz="0.0" izz="0.0"/>
+               </inertial>
+               <visual name="">
+                    <origin xyz="0.0 0.0 0.0" rpy="0.0 0.0 0.0"/>
+                    <geometry>
+                         <mesh filename="package://robot_simulation_description/meshes/Kinect.dae" scale="0.0010 0.0010 0.0010"/>
+                    </geometry>
+                    <material name="">
+                         <color rgba="0.0 0.0 0.0 1.0"/>
+                         <texture filename=""/>
+                    </material>
+               </visual>
+               <collision>
+                    <origin xyz="0.0 0.0 0.0" rpy="0.0 0.0 0.0"/>
+                    <geometry>
+                         <mesh filename="package://robot_simulation_description/meshes/Kinect.dae" scale="0.0010 0.0010 0.0010"/>
+                    </geometry>
+               </collision>
+          </link>
+          <joint name="camera_joint" type="fixed">
+               <origin xyz="0.30 0.0 0.06" rpy="0.0 0.0 1.5705"/>
+               <parent link="base_link"/>
+               <child link="camera_link"/>
+               <axis xyz="0.0 0.0 0.0"/>
+          </joint>
+          <!---LiDAR Camera-->
+          <link name="LiDAR_link">
+               <inertial>
+                    <origin xyz="0.0 0.0 0.0" rpy="0.0 0.0 0.0"/>
+                    <mass value="0.1"/>
+                    <inertia ixx="0.0" ixy="0.0" ixz="0.0" iyy="0.0" iyz="0.0" izz="0.0"/>
+               </inertial>
+               <visual name="">
+                    <origin xyz="0.0 0.0 0.0" rpy="0.0 0.0 0.0"/>
+                    <geometry>
+                         <mesh filename="package://robot_simulation_description/meshes/LiDAR.dae" scale="0.0015 0.0015 0.0015"/>
+                    </geometry>
+                    <material name="black">
+                         <color rgba="0.0 0.0 0.0 1.0"/>
+                         <texture filename=""/>
+                    </material>
+               </visual>
+               <collision>
+                    <origin xyz="0.0 0.0 0.0" rpy="0.0 0.0 0.0"/>
+                    <geometry>
+                         <mesh filename="package://robot_simulation_description/meshes/LiDAR.dae" scale="0.0015 0.0015 0.0015"/>
+                    </geometry>
+               </collision>
+          </link>
+          <joint name="LiDAR_joint" type="fixed">
+               <origin xyz="0.26 -0.06 -0.00" rpy="1.5705 0 3.14"/>
+               <parent link="top_layer_link"/>
+               <child link="LiDAR_link"/>
+               <axis xyz="0.0 0.0 0.0"/>
+          </joint>
 </robot>

Commit message: Adding the Kinect/depth camera plugin to Gazebo

File: urdf/rabe_bot_basic.urdf.xacro (robot description, xacro)
@@ -212,4 +212,13 @@
                <axis xyz="0.0 0.0 0.0"/>
           </joint>
+          <!-- For Optical data correction if needed .. -->
+          <link name="camera_optical_data_correction_link">
+          </link>
+          <joint name="camera_optical_data_correction_joint" type="fixed">
+               <origin xyz="0.0 0.0 0.0" rpy="0.0 0.0 -1.5705"/>
+               <parent link="camera_link"/>
+               <child link="camera_optical_data_correction_link"/>
+               <axis xyz="0.0 0.0 0.0"/>
+          </joint>
           <!---LiDAR Camera-->
           <link name="LiDAR_link">
@@ -242,3 +251,12 @@
                <axis xyz="0.0 0.0 0.0"/>
           </joint>
+          <!-- For LiDAR data correction if needed .. -->
+          <link name="LiDAR_optical_data_correction_link">
+          </link>
+          <joint name="LiDAR_optical_data_correction_joint" type="fixed">
+               <origin xyz="0.0 0.0 0.0" rpy="0.0 0.0 0.0"/>
+               <parent link="LiDAR_link"/>
+               <child link="LiDAR_optical_data_correction_link"/>
+               <axis xyz="0.0 0.0 0.0"/>
+          </joint>
 </robot>

Commit message: adding the Lidar plugin

File: urdf/rabe_bot_basic.urdf.xacro (robot description, xacro)
@@ -54,5 +54,5 @@
                                         <origin xyz="0.0 0.0 0.0" rpy="0.0 0.0 0.0"/>
                                         <geometry>
-                                                  <cylinder radius="0.015" length="0.2"/>
+                                                  <cylinder radius="${radius}" length="${length}"/>
                                         </geometry>
                                         <material name="">
@@ -64,5 +64,5 @@
                                         <origin xyz="0.0 0.0 0.0" rpy="0.0 0.0 0.0"/>
                                         <geometry>
-                                                  <cylinder radius="0.015" length="0.2"/>
+                                                  <cylinder radius="${radius}" length="${length}"/>
                                         </geometry>
                               </collision>
@@ -80,4 +80,5 @@
           <xacro:stand name="rear_right_stand" x="0.25" y="-0.15" z="0.1" mass="0.05" radius="0.015" length="0.2"/>
           <xacro:stand name="rear_left_stand" x="0.25" y="0.15" z="0.1" mass="0.05" radius="0.015" length="0.2"/>
+          <xacro:stand name="under_lidar_stand" x="0.2" y="-0.0" z="0.30" mass="0.05" radius="0.03" length="0.15"/>
           <!-- Layer Two Top -->
           <link name="top_layer_link">
@@ -182,5 +183,5 @@
 <xacro:wheel_right name="rear_right_wheel" x="-0.2" y="-0.26"/>
 <xacro:wheel_left name="rear_left_wheel" x="-0.2" y="0.26"/>
-          <!---Kinect/Depth Camera-->
+          <!---Kinect/Depth Camera  POINTCLOUD-->
           <link name="camera_link">
                <inertial>
@@ -221,6 +222,6 @@
                <axis xyz="0.0 0.0 0.0"/>
           </joint>
-          <!---LiDAR Camera-->
-          <link name="LiDAR_link">
+         <!---LiDAR Camera-->
+          <link name="lidar_link">
                <inertial>
                     <origin xyz="0.0 0.0 0.0" rpy="0.0 0.0 0.0"/>
@@ -228,5 +229,5 @@
                     <inertia ixx="0.0" ixy="0.0" ixz="0.0" iyy="0.0" iyz="0.0" izz="0.0"/>
                </inertial>
-               <visual name="">
+               <visual name="lidar_visual">
                     <origin xyz="0.0 0.0 0.0" rpy="0.0 0.0 0.0"/>
                     <geometry>
@@ -245,17 +246,18 @@
                </collision>
           </link>
-          <joint name="LiDAR_joint" type="fixed">
-               <origin xyz="0.26 -0.06 -0.00" rpy="1.5705 0 3.14"/>
+          <joint name="lidar_joint" type="fixed">
+               <!-- <origin xyz="0.26 -0.06 0.00" rpy="1.5705 0 3.14"/> -->
+               <origin xyz="0.26 -0.05 0.15" rpy="1.5705 0 3.14"/>
                <parent link="top_layer_link"/>
-               <child link="LiDAR_link"/>
+               <child link="lidar_link"/>
                <axis xyz="0.0 0.0 0.0"/>
           </joint>
           <!-- For LiDAR data correction if needed .. -->
-          <link name="LiDAR_optical_data_correction_link">
-          </link>
-          <joint name="LiDAR_optical_data_correction_joint" type="fixed">
-               <origin xyz="0.0 0.0 0.0" rpy="0.0 0.0 0.0"/>
-               <parent link="LiDAR_link"/>
-               <child link="LiDAR_optical_data_correction_link"/>
+          <link name="lidar_optical_data_correction_link">
+          </link>
+          <joint name="lidar_optical_data_correction_joint" type="fixed">
+               <origin xyz="0.0 0.0 0.0" rpy="1.5705 0.0 0.0"/>
+               <parent link="lidar_link"/>
+               <child link="lidar_optical_data_correction_link"/>
                <axis xyz="0.0 0.0 0.0"/>
           </joint>
